File: hardware/boards/glasgow/glasgow.kicad_pcb (KiCad board)
At the start: 4 copper layers, 80 x 49 mm, 240 parts, among them J1 USB_B_Micro, J10 Conn_01x03, J2 Conn_02x10_Odd_Even, J3 Conn_02x10_Odd_Even, J4 Conn_01x02, J5 Conn_02x22_Odd_Even, J6 Conn_01x08, J7 Conn_01x08, J8 Conn_01x08, J9 Conn_01x08, U1 CY7C68013A-56LTX, U10 SN74LVC1T45DRL, U11 SN74LVC1T45DRL, U12 ADC081C021CIMM, U13 DAC081C081CIMK, U14 TPS73101DBV, U15 TPD3S014, U16 SN74LVC1T45DRL, U17 SN74LVC1T45DRL, U18 SN74LVC1T45DRL, U19 PCA6408APW, U2 CAT24M01W, U20 DAC081C081CIMK, U21 ADC081C021CIMM, U22 SN74LVC1T45DRL, U23 SN74LVC1T45DRL, U24 SN74LVC1T45DRL, U25 SN74LVC1T45DRL, U26 SN74LVC1T45DRL, U27 SN74LVC1T45DRL, U28 SN74LVC1T45DRL, U29 SN74LVC1T45DRL, U3 CAT24C256W, U30 ICE40HX8K-BG121, U31 TPS73101DBV, U32 SN74LVC1T45DRL, U33 MG2040, U34 ATECC508A, U35 MG2040, U36 TLV73312PQDRVRQ1, U4 SN74LVC1T45DRL, U5 PCA6408APW, U6 SN74LVC1T45DRL, U7 LM3880MF-1AF, U8 TLV75533PDRVR, U9 SN74LVC1T45DRL, Y1 24M

Commit message: revC2: added output files
Parts:
- added R52: 5k1, Resistor_SMD:R_0402_1005Metric, F.Cu at (53.6, 90.2)
- added R53: 5k1, Resistor_SMD:R_0402_1005Metric, F.Cu at (53.6, 100.8)
- J1: value USB_B_Micro -> USB_C_Plug_USB2.0; footprint Connector_USB:USB_Micro-B_Molex_47346-0001 -> Glasgow:USB-C_16Pin
- moved C13 10.3 mm to (58.5, 91.0)
- moved R3 10.3 mm to (58.5, 90.0)
- moved J1 2.70 mm to (56.5, 95.5)
- moved FB1 0.73 mm to (58.4, 94.2), turned to 270 degrees
- moved TP13 0.66 mm to (56.1, 93.2)
- moved TP14 0.66 mm to (56.1, 97.7)
- moved TP15 0.66 mm to (56.1, 96.2)
- moved TP16 0.66 mm to (56.1, 94.7)
- moved C11 0.32 mm to (61.9, 90.2)
- moved C12 0.32 mm to (61.9, 95.0)
- moved Y1 0.32 mm to (61.9, 92.6)
Routing:
- net Net-(FB1-Pad1): track 3.71 -> 12.2 mm
- net Net-(J1-PadA5): track 0.00 -> 7.59 mm, vias 0 -> 2
- net Net-(J1-PadB5): track 0.00 -> 7.46 mm, vias 0 -> 2
- net /SHLD: track 15.1 -> 20.4 mm
- net GND: track 262.0 -> 266.1 mm
- net /VUSB: track 9.50 -> 8.69 mm
- net /USB_P: track 18.9 -> 18.8 mm, vias 2 -> 1
Other:
- outline, holes or cut-outs redrawn
- board text added: "Glasgow revC2"
- board text removed: "Glasgow revC1"

Commit message: added revC1 otter edition gerber
Parts:
- added G***: LOGO, otter:kicad_designer_84, B.Cu at (66.8, 115.7)
- J1: value USB_C_Plug_USB2.0 -> USB; footprint Glasgow:USB-C_16Pin -> otter:USB-C 16Pin
- moved J1 0.15 mm to (56.4, 95.5)
Connections:
- J1 pad A8: (no net) -> Net-(J1-PadA8)
- J1 pad B6: (no net) -> /USB_P
- J1 pad B7: (no net) -> /USB_N
- J1 pad B8: (no net) -> Net-(J1-PadB8)
Routing:
- net /USB_P: track 18.8 -> 21.7 mm, vias 1 -> 2
- net /USB_N: track 18.7 -> 20.6 mm
- net /SHLD: track 20.4 -> 22.1 mm
